Commit message: Face table: rotate base in observation pose, tilt camera more

File: color_sorting_arm/urdf/arm.urdf.xacro (robot description, xacro)
@@ -287,5 +287,5 @@
     <child link="camera_link"/>
     <!-- Move camera forward/up and tilt it down to face the table -->
-    <origin xyz="0.07 0 0.05" rpy="0 -1.3 0"/>
+    <origin xyz="0.09 0 0.07" rpy="0 -1.45 0"/>
   </joint>
   <!-- Camera Optical Frame -->
