Commit message: Fix arm design: shorter links, separate camera, test movements on startup
- Redesigned arm URDF with shorter link lengths for better proportions
- Camera now in world file as separate overhead stand (not attached to arm)
- Camera positioned to see entire table from above
- Added startup test movements in sorting_controller
- Created test_arm_movement.py for manual arm testing
- Cubes placed in random positions on table
- Updated camera topics to /camera/image_raw
- Updated IK parameters to match new arm dimensions

File: color_sorting_arm/urdf/arm.gazebo.xacro (robot description, xacro)
@@ -44,47 +44,5 @@
     <mu2>1.5</mu2>
   </gazebo>
-  <gazebo reference="camera_pole">
-    <material>Gazebo/Grey</material>
-  </gazebo>
-  <gazebo reference="camera_link">
-    <material>Gazebo/DarkGrey</material>
-  </gazebo>
-  <!-- Camera sensor plugin -->
-  <gazebo reference="camera_link">
-    <sensor type="camera" name="camera1">
-      <update_rate>30.0</update_rate>
-      <camera name="head">
-        <horizontal_fov>1.3962634</horizontal_fov>
-        <image>
-          <width>640</width>
-          <height>480</height>
-          <format>R8G8B8</format>
-        </image>
-        <clip>
-          <near>0.02</near>
-          <far>300</far>
-        </clip>
-        <noise>
-          <type>gaussian</type>
-          <mean>0.0</mean>
-          <stddev>0.007</stddev>
-        </noise>
-      </camera>
-      <plugin name="camera_controller" filename="libgazebo_ros_camera.so">
-        <alwaysOn>true</alwaysOn>
-        <updateRate>0.0</updateRate>
-        <cameraName>arm_camera</cameraName>
-        <imageTopicName>image_raw</imageTopicName>
-        <cameraInfoTopicName>camera_info</cameraInfoTopicName>
-        <frameName>camera_optical_frame</frameName>
-        <hackBaseline>0.07</hackBaseline>
-        <distortionK1>0.0</distortionK1>
-        <distortionK2>0.0</distortionK2>
-        <distortionK3>0.0</distortionK3>
-        <distortionT1>0.0</distortionT1>
-        <distortionT2>0.0</distortionT2>
-      </plugin>
-    </sensor>
-  </gazebo>
+  <!-- Camera is now separate - see camera_stand.urdf.xacro -->
   <!-- Transmissions for ros_control -->
   <transmission name="trans_joint1">

File: color_sorting_arm/urdf/arm.urdf.xacro (robot description, xacro)
@@ -22,20 +22,20 @@
   <link name="base_link">
     <visual>
-      <origin xyz="0 0 0.025" rpy="0 0 0"/>
-      <geometry>
-        <cylinder radius="0.08" length="0.05"/>
+      <origin xyz="0 0 0.02" rpy="0 0 0"/>
+      <geometry>
+        <cylinder radius="0.06" length="0.04"/>
       </geometry>
       <material name="dark_grey"/>
     </visual>
     <collision>
-      <origin xyz="0 0 0.025" rpy="0 0 0"/>
-      <geometry>
-        <cylinder radius="0.08" length="0.05"/>
-      </geometry>
-    </collision>
-    <inertial>
-      <origin xyz="0 0 0.025" rpy="0 0 0"/>
-      <mass value="2.0"/>
-      <inertia ixx="0.005" ixy="0" ixz="0" iyy="0.005" iyz="0" izz="0.005"/>
+      <origin xyz="0 0 0.02" rpy="0 0 0"/>
+      <geometry>
+        <cylinder radius="0.06" length="0.04"/>
+      </geometry>
+    </collision>
+    <inertial>
+      <origin xyz="0 0 0.02" rpy="0 0 0"/>
+      <mass value="1.0"/>
+      <inertia ixx="0.002" ixy="0" ixz="0" iyy="0.002" iyz="0" izz="0.002"/>
     </inertial>
   </link>
@@ -43,20 +43,20 @@
   <link name="link1">
     <visual>
-      <origin xyz="0 0 0.04" rpy="0 0 0"/>
-      <geometry>
-        <cylinder radius="0.045" length="0.08"/>
+      <origin xyz="0 0 0.025" rpy="0 0 0"/>
+      <geometry>
+        <cylinder radius="0.035" length="0.05"/>
       </geometry>
       <material name="orange"/>
     </visual>
     <collision>
-      <origin xyz="0 0 0.04" rpy="0 0 0"/>
-      <geometry>
-        <cylinder radius="0.045" length="0.08"/>
-      </geometry>
-    </collision>
-    <inertial>
-      <origin xyz="0 0 0.04" rpy="0 0 0"/>
-      <mass value="0.5"/>
-      <inertia ixx="0.001" ixy="0" ixz="0" iyy="0.001" iyz="0" izz="0.0005"/>
+      <origin xyz="0 0 0.025" rpy="0 0 0"/>
+      <geometry>
+        <cylinder radius="0.035" length="0.05"/>
+      </geometry>
+    </collision>
+    <inertial>
+      <origin xyz="0 0 0.025" rpy="0 0 0"/>
+      <mass value="0.3"/>
+      <inertia ixx="0.0005" ixy="0" ixz="0" iyy="0.0005" iyz="0" izz="0.0003"/>
     </inertial>
   </link>
@@ -64,5 +64,5 @@
     <parent link="base_link"/>
     <child link="link1"/>
-    <origin xyz="0 0 0.05" rpy="0 0 0"/>
+    <origin xyz="0 0 0.04" rpy="0 0 0"/>
     <axis xyz="0 0 1"/>
     <limit lower="${-PI}" upper="${PI}" effort="30" velocity="1.5"/>
@@ -72,20 +72,20 @@
   <link name="link2">
     <visual>
-      <origin xyz="0 0 0.075" rpy="0 0 0"/>
-      <geometry>
-        <box size="0.05 0.05 0.15"/>
+      <origin xyz="0 0 0.04" rpy="0 0 0"/>
+      <geometry>
+        <box size="0.03 0.03 0.08"/>
       </geometry>
       <material name="blue"/>
     </visual>
     <collision>
-      <origin xyz="0 0 0.075" rpy="0 0 0"/>
-      <geometry>
-        <box size="0.05 0.05 0.15"/>
-      </geometry>
-    </collision>
-    <inertial>
-      <origin xyz="0 0 0.075" rpy="0 0 0"/>
-      <mass value="0.4"/>
-      <inertia ixx="0.001" ixy="0" ixz="0" iyy="0.001" iyz="0" izz="0.0003"/>
+      <origin xyz="0 0 0.04" rpy="0 0 0"/>
+      <geometry>
+        <box size="0.03 0.03 0.08"/>
+      </geometry>
+    </collision>
+    <inertial>
+      <origin xyz="0 0 0.04" rpy="0 0 0"/>
+      <mass value="0.2"/>
+      <inertia ixx="0.0003" ixy="0" ixz="0" iyy="0.0003" iyz="0" izz="0.0001"/>
     </inertial>
   </link>
@@ -93,5 +93,5 @@
     <parent link="link1"/>
     <child link="link2"/>
-    <origin xyz="0 0 0.08" rpy="0 0 0"/>
+    <origin xyz="0 0 0.05" rpy="0 0 0"/>
     <axis xyz="0 1 0"/>
     <limit lower="${-PI/2}" upper="${PI/2}" effort="30" velocity="1.5"/>
@@ -101,20 +101,20 @@
   <link name="link3">
     <visual>
-      <origin xyz="0 0 0.075" rpy="0 0 0"/>
-      <geometry>
-        <box size="0.04 0.04 0.15"/>
+      <origin xyz="0 0 0.035" rpy="0 0 0"/>
+      <geometry>
+        <box size="0.025 0.025 0.07"/>
       </geometry>
       <material name="white"/>
     </visual>
     <collision>
-      <origin xyz="0 0 0.075" rpy="0 0 0"/>
-      <geometry>
-        <box size="0.04 0.04 0.15"/>
-      </geometry>
-    </collision>
-    <inertial>
-      <origin xyz="0 0 0.075" rpy="0 0 0"/>
-      <mass value="0.3"/>
-      <inertia ixx="0.0008" ixy="0" ixz="0" iyy="0.0008" iyz="0" izz="0.0002"/>
+      <origin xyz="0 0 0.035" rpy="0 0 0"/>
+      <geometry>
+        <box size="0.025 0.025 0.07"/>
+      </geometry>
+    </collision>
+    <inertial>
+      <origin xyz="0 0 0.035" rpy="0 0 0"/>
+      <mass value="0.15"/>
+      <inertia ixx="0.0002" ixy="0" ixz="0" iyy="0.0002" iyz="0" izz="0.00005"/>
     </inertial>
   </link>
@@ -122,28 +122,28 @@
     <parent link="link2"/>
     <child link="link3"/>
-    <origin xyz="0 0 0.15" rpy="0 0 0"/>
+    <origin xyz="0 0 0.08" rpy="0 0 0"/>
     <axis xyz="0 1 0"/>
     <limit lower="${-2.5}" upper="${2.5}" effort="20" velocity="1.5"/>
     <dynamics damping="0.3" friction="0.1"/>
   </joint>
-  <!-- ===================== LINK 4 - WRIST PITCH ===================== -->
+  <!-- ===================== LINK 4 - WRIST ===================== -->
   <link name="link4">
     <visual>
-      <origin xyz="0 0 0.04" rpy="0 0 0"/>
-      <geometry>
-        <box size="0.035 0.035 0.08"/>
+      <origin xyz="0 0 0.025" rpy="0 0 0"/>
+      <geometry>
+        <box size="0.02 0.02 0.05"/>
       </geometry>
       <material name="blue"/>
     </visual>
     <collision>
-      <origin xyz="0 0 0.04" rpy="0 0 0"/>
-      <geometry>
-        <box size="0.035 0.035 0.08"/>
-      </geometry>
-    </collision>
-    <inertial>
-      <origin xyz="0 0 0.04" rpy="0 0 0"/>
-      <mass value="0.15"/>
-      <inertia ixx="0.0003" ixy="0" ixz="0" iyy="0.0003" iyz="0" izz="0.0001"/>
+      <origin xyz="0 0 0.025" rpy="0 0 0"/>
+      <geometry>
+        <box size="0.02 0.02 0.05"/>
+      </geometry>
+    </collision>
+    <inertial>
+      <origin xyz="0 0 0.025" rpy="0 0 0"/>
+      <mass value="0.1"/>
+      <inertia ixx="0.0001" ixy="0" ixz="0" iyy="0.0001" iyz="0" izz="0.00005"/>
     </inertial>
   </link>
@@ -151,5 +151,5 @@
     <parent link="link3"/>
     <child link="link4"/>
-    <origin xyz="0 0 0.15" rpy="0 0 0"/>
+    <origin xyz="0 0 0.07" rpy="0 0 0"/>
     <axis xyz="0 1 0"/>
     <limit lower="${-PI/2}" upper="${PI/2}" effort="10" velocity="2.0"/>
@@ -159,20 +159,20 @@
   <link name="link5">
     <visual>
-      <origin xyz="0 0 0.02" rpy="0 0 0"/>
-      <geometry>
-        <cylinder radius="0.02" length="0.04"/>
+      <origin xyz="0 0 0.015" rpy="0 0 0"/>
+      <geometry>
+        <cylinder radius="0.015" length="0.03"/>
       </geometry>
       <material name="white"/>
     </visual>
     <collision>
-      <origin xyz="0 0 0.02" rpy="0 0 0"/>
-      <geometry>
-        <cylinder radius="0.02" length="0.04"/>
-      </geometry>
-    </collision>
-    <inertial>
-      <origin xyz="0 0 0.02" rpy="0 0 0"/>
-      <mass value="0.08"/>
-      <inertia ixx="0.00005" ixy="0" ixz="0" iyy="0.00005" iyz="0" izz="0.00002"/>
+      <origin xyz="0 0 0.015" rpy="0 0 0"/>
+      <geometry>
+        <cylinder radius="0.015" length="0.03"/>
+      </geometry>
+    </collision>
+    <inertial>
+      <origin xyz="0 0 0.015" rpy="0 0 0"/>
+      <mass value="0.05"/>
+      <inertia ixx="0.00002" ixy="0" ixz="0" iyy="0.00002" iyz="0" izz="0.00001"/>
     </inertial>
   </link>
@@ -180,5 +180,5 @@
     <parent link="link4"/>
     <child link="link5"/>
-    <origin xyz="0 0 0.08" rpy="0 0 0"/>
+    <origin xyz="0 0 0.05" rpy="0 0 0"/>
     <axis xyz="0 0 1"/>
     <limit lower="${-PI}" upper="${PI}" effort="5" velocity="2.0"/>
@@ -188,20 +188,20 @@
   <link name="gripper_base">
     <visual>
-      <origin xyz="0 0 0.015" rpy="0 0 0"/>
-      <geometry>
-        <box size="0.03 0.06 0.03"/>
+      <origin xyz="0 0 0.01" rpy="0 0 0"/>
+      <geometry>
+        <box size="0.02 0.04 0.02"/>
       </geometry>
       <material name="grey"/>
     </visual>
     <collision>
-      <origin xyz="0 0 0.015" rpy="0 0 0"/>
-      <geometry>
-        <box size="0.03 0.06 0.03"/>
-      </geometry>
-    </collision>
-    <inertial>
-      <origin xyz="0 0 0.015" rpy="0 0 0"/>
-      <mass value="0.05"/>
-      <inertia ixx="0.00002" ixy="0" ixz="0" iyy="0.00002" iyz="0" izz="0.00002"/>
+      <origin xyz="0 0 0.01" rpy="0 0 0"/>
+      <geometry>
+        <box size="0.02 0.04 0.02"/>
+      </geometry>
+    </collision>
+    <inertial>
+      <origin xyz="0 0 0.01" rpy="0 0 0"/>
+      <mass value="0.03"/>
+      <inertia ixx="0.00001" ixy="0" ixz="0" iyy="0.00001" iyz="0" izz="0.00001"/>
     </inertial>
   </link>
@@ -209,25 +209,25 @@
     <parent link="link5"/>
     <child link="gripper_base"/>
-    <origin xyz="0 0 0.04" rpy="0 0 0"/>
+    <origin xyz="0 0 0.03" rpy="0 0 0"/>
   </joint>
   <!-- ===================== LEFT FINGER ===================== -->
   <link name="gripper_left">
     <visual>
-      <origin xyz="0 0 0.025" rpy="0 0 0"/>
-      <geometry>
-        <box size="0.01 0.015 0.05"/>
+      <origin xyz="0 0 0.02" rpy="0 0 0"/>
+      <geometry>
+        <box size="0.008 0.01 0.04"/>
       </geometry>
       <material name="dark_grey"/>
     </visual>
     <collision>
-      <origin xyz="0 0 0.025" rpy="0 0 0"/>
-      <geometry>
-        <box size="0.01 0.015 0.05"/>
-      </geometry>
-    </collision>
-    <inertial>
-      <origin xyz="0 0 0.025" rpy="0 0 0"/>
-      <mass value="0.02"/>
-      <inertia ixx="0.000005" ixy="0" ixz="0" iyy="0.000005" iyz="0" izz="0.000002"/>
+      <origin xyz="0 0 0.02" rpy="0 0 0"/>
+      <geometry>
+        <box size="0.008 0.01 0.04"/>
+      </geometry>
+    </collision>
+    <inertial>
+      <origin xyz="0 0 0.02" rpy="0 0 0"/>
+      <mass value="0.01"/>
+      <inertia ixx="0.000002" ixy="0" ixz="0" iyy="0.000002" iyz="0" izz="0.000001"/>
     </inertial>
   </link>
@@ -235,7 +235,7 @@
     <parent link="gripper_base"/>
     <child link="gripper_left"/>
-    <origin xyz="0 0.015 0.03" rpy="0 0 0"/>
-    <axis xyz="0 1 0"/>
-    <limit lower="0" upper="0.02" effort="5" velocity="0.1"/>
+    <origin xyz="0 0.012 0.02" rpy="0 0 0"/>
+    <axis xyz="0 1 0"/>
+    <limit lower="0" upper="0.015" effort="5" velocity="0.1"/>
     <dynamics damping="0.5"/>
   </joint>
@@ -243,20 +243,20 @@
   <link name="gripper_right">
     <visual>
-      <origin xyz="0 0 0.025" rpy="0 0 0"/>
-      <geometry>
-        <box size="0.01 0.015 0.05"/>
+      <origin xyz="0 0 0.02" rpy="0 0 0"/>
+      <geometry>
+        <box size="0.008 0.01 0.04"/>
       </geometry>
       <material name="dark_grey"/>
     </visual>
     <collision>
-      <origin xyz="0 0 0.025" rpy="0 0 0"/>
-      <geometry>
-        <box size="0.01 0.015 0.05"/>
-      </geometry>
-    </collision>
-    <inertial>
-      <origin xyz="0 0 0.025" rpy="0 0 0"/>
-      <mass value="0.02"/>
-      <inertia ixx="0.000005" ixy="0" ixz="0" iyy="0.000005" iyz="0" izz="0.000002"/>
+      <origin xyz="0 0 0.02" rpy="0 0 0"/>
+      <geometry>
+        <box size="0.008 0.01 0.04"/>
+      </geometry>
+    </collision>
+    <inertial>
+      <origin xyz="0 0 0.02" rpy="0 0 0"/>
+      <mass value="0.01"/>
+      <inertia ixx="0.000002" ixy="0" ixz="0" iyy="0.000002" iyz="0" izz="0.000001"/>
     </inertial>
   </link>
@@ -264,67 +264,8 @@
     <parent link="gripper_base"/>
     <child link="gripper_right"/>
-    <origin xyz="0 -0.015 0.03" rpy="0 0 0"/>
+    <origin xyz="0 -0.012 0.02" rpy="0 0 0"/>
     <axis xyz="0 -1 0"/>
-    <limit lower="0" upper="0.02" effort="5" velocity="0.1"/>
+    <limit lower="0" upper="0.015" effort="5" velocity="0.1"/>
     <dynamics damping="0.5"/>
   </joint>
-  <!-- ===================== CAMERA - FIXED ON POLE ===================== -->
-  <!-- Camera mounted on a separate pole/stand looking down at workspace -->
-  <link name="camera_pole">
-    <visual>
-      <origin xyz="0 0 0.15" rpy="0 0 0"/>
-      <geometry>
-        <cylinder radius="0.015" length="0.3"/>
-      </geometry>
-      <material name="grey"/>
-    </visual>
-    <collision>
-      <origin xyz="0 0 0.15" rpy="0 0 0"/>
-      <geometry>
-        <cylinder radius="0.015" length="0.3"/>
-      </geometry>
-    </collision>
-    <inertial>
-      <origin xyz="0 0 0.15" rpy="0 0 0"/>
-      <mass value="0.2"/>
-      <inertia ixx="0.002" ixy="0" ixz="0" iyy="0.002" iyz="0" izz="0.0001"/>
-    </inertial>
-  </link>
-  <joint name="camera_pole_joint" type="fixed">
-    <parent link="base_link"/>
-    <child link="camera_pole"/>
-    <origin xyz="-0.15 0 0.05" rpy="0 0 0"/>
-  </joint>
-  <link name="camera_link">
-    <visual>
-      <origin xyz="0 0 0" rpy="0 0 0"/>
-      <geometry>
-        <box size="0.04 0.06 0.03"/>
-      </geometry>
-      <material name="dark_grey"/>
-    </visual>
-    <collision>
-      <origin xyz="0 0 0" rpy="0 0 0"/>
-      <geometry>
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